File: eagle/esp8266-rfid.brd (EAGLE design)
At the start: 41 x 49 mm, 18 parts, among them J1 USB-MICROB", U1 esp-12

Commit message: EAGLE moved to new folder
Routing:
- net RX: track 35.9 -> 72.9 mm
Changed lines of the file:
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@@
 <layer number="14" name="Route14" color="1" fill="6" visible="no" active="no"/>
 <layer number="15" name="Route15" color="4" fill="6" visible="no" active="no"/>
-<layer number="16" name="Bottom" color="1" fill="1" visible="yes" active="yes"/>
+<layer number="16" name="Bottom" color="1" fill="1" visible="no" active="yes"/>
 <layer number="17" name="Pads" color="2" fill="1" visible="yes" active="yes"/>
 <layer number="18" name="Vias" color="2" fill="1" visible="yes" active="yes"/>
@@
 <via x="3.335934375" y="39.769640625" extent="1-16" drill="0.3048"/>
 <via x="36.593753125" y="36.133278125" extent="1-16" drill="0.3048"/>
-<via x="32.967590625" y="15.4788875" extent="1-16" drill="0.3048"/>
+<via x="31.967590625" y="17.4788875" extent="1-16" drill="0.3048"/>
 <via x="35.4718625" y="25.88095" extent="1-16" drill="0.3048"/>
 <via x="30.29856875" y="2.900325" extent="1-16" drill="0.3048"/>
@@
 <wire x1="22.1" y1="44.4" x2="21.465" y2="43.765" width="0.254" layer="1"/>
 <wire x1="21.465" y1="43.765" x2="21.465" y2="42.83" width="0.254" layer="1"/>
-<wire x1="17.6" y1="11.4" x2="21.465" y2="42.83" width="0" layer="19" extent="16-16"/>
+<wire x1="33.508" y1="44.092" x2="33.508" y2="7.112" width="0.254" layer="1"/>
 </signal>
 </signals>

Commit message: EAGLE + http push
Connections:
- removed net +5V: U$1.11, U$1.2
- removed net N$3: J1.VBUS, T1.3
- new net VBUS: J1.VBUS, T1.3, U$1.11, U$1.2
Routing:
- net VBUS: track 0.00 -> 63.1 mm, vias 0 -> 2
- net N$3: track 21.3 -> 0.00 mm, vias 1 -> 0
- net +5V: track 19.8 -> 0.00 mm
Changed lines of the file:
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@@
 <layer number="14" name="Route14" color="1" fill="6" visible="no" active="no"/>
 <layer number="15" name="Route15" color="4" fill="6" visible="no" active="no"/>
-<layer number="16" name="Bottom" color="1" fill="1" visible="no" active="yes"/>
+<layer number="16" name="Bottom" color="1" fill="1" visible="yes" active="yes"/>
 <layer number="17" name="Pads" color="2" fill="1" visible="yes" active="yes"/>
 <layer number="18" name="Vias" color="2" fill="1" visible="yes" active="yes"/>
-<layer number="19" name="Unrouted" color="6" fill="1" visible="no" active="yes"/>
+<layer number="19" name="Unrouted" color="6" fill="1" visible="yes" active="yes"/>
 <layer number="20" name="Dimension" color="15" fill="1" visible="yes" active="yes"/>
 <layer number="21" name="tPlace" color="7" fill="1" visible="yes" active="yes"/>
@@
 <via x="3.599309375" y="11.4291625" extent="1-16" drill="0.3048"/>
 </signal>
-<signal name="+5V">
-<contactref element="U$1" pad="11"/>
-<contactref element="U$1" pad="2"/>
-<wire x1="27.465" y1="42.83" x2="27.465" y2="33.765" width="0.254" layer="1"/>
-<wire x1="27.465" y1="33.765" x2="27" y2="33.3" width="0.254" layer="1"/>
-<wire x1="27" y1="33.3" x2="23" y2="33.3" width="0.254" layer="1"/>
-<wire x1="23" y1="33.3" x2="21.465" y2="31.765" width="0.254" layer="1"/>
-<wire x1="21.465" y1="31.765" x2="21.465" y2="27.83" width="0.254" layer="1"/>
-</signal>
 <signal name="N$7">
 <contactref element="U1" pad="GPIO4"/>
@@
 <wire x1="24.77" y1="5.6" x2="24.824" y2="5.654" width="0.254" layer="1"/>
 </signal>
-<signal name="N$3">
-<contactref element="J1" pad="VBUS"/>
-<contactref element="T1" pad="3"/>
-<wire x1="19" y1="6.4" x2="21.2" y2="4.2" width="0.254" layer="16"/>
-<wire x1="21.2" y1="4.2" x2="26" y2="4.2" width="0.254" layer="16"/>
-<wire x1="26" y1="4.2" x2="26.6" y2="4.8" width="0.254" layer="16"/>
-<wire x1="26.6" y1="4.8" x2="26.6" y2="12" width="0.254" layer="16"/>
-<via x="26.6" y="12" extent="1-16" drill="0.3048"/>
-<wire x1="26.6" y1="12" x2="26.6" y2="13.7" width="0.254" layer="1"/>
-<wire x1="26.6" y1="13.7" x2="26.743" y2="13.843" width="0.254" layer="1"/>
-<wire x1="19" y1="6.4" x2="16.7" y2="6.4" width="0.254" layer="16"/>
-<wire x1="16.7" y1="6.4" x2="16.436" y2="6.136" width="0.254" layer="16"/>
-<wire x1="16.436" y1="6.136" x2="16.436" y2="5.417" width="0.254" layer="16"/>
-</signal>
 <signal name="N$8">
 <contactref element="U1" pad="VCC"/>
@@
 <wire x1="33.508" y1="44.092" x2="33.508" y2="7.112" width="0.254" layer="1"/>
 </signal>
+<signal name="VBUS">
+<contactref element="U$1" pad="2"/>
+<contactref element="J1" pad="VBUS"/>
+<contactref element="T1" pad="3"/>
+<wire x1="19" y1="6.4" x2="21.2" y2="4.2" width="0.254" layer="16"/>
+<wire x1="21.2" y1="4.2" x2="26" y2="4.2" width="0.254" layer="16"/>
+<wire x1="26" y1="4.2" x2="26.6" y2="4.8" width="0.254" layer="16"/>
+<wire x1="26.6" y1="4.8" x2="26.6" y2="12" width="0.254" layer="16"/>
+<via x="26.6" y="12" extent="1-16" drill="0.3048"/>
+<wire x1="26.6" y1="12" x2="26.6" y2="13.7" width="0.254" layer="1"/>
+<wire x1="26.6" y1="13.7" x2="26.743" y2="13.843" width="0.254" layer="1"/>
+<wire x1="19" y1="6.4" x2="16.7" y2="6.4" width="0.254" layer="16"/>
+<wire x1="16.7" y1="6.4" x2="16.436" y2="6.136" width="0.254" layer="16"/>
+<wire x1="16.436" y1="6.136" x2="16.436" y2="5.417" width="0.254" layer="16"/>
+<contactref element="U$1" pad="11"/>
+<wire x1="27.465" y1="42.83" x2="27.465" y2="33.765" width="0.254" layer="1"/>
+<wire x1="27.465" y1="33.765" x2="27" y2="33.3" width="0.254" layer="1"/>
+<wire x1="27" y1="33.3" x2="23" y2="33.3" width="0.254" layer="1"/>
+<wire x1="23" y1="33.3" x2="21.465" y2="31.765" width="0.254" layer="1"/>
+<wire x1="21.465" y1="31.765" x2="21.465" y2="27.83" width="0.4064" layer="1"/>
+<wire x1="21.465" y1="27.83" x2="21.465" y2="25.535" width="0.4064" layer="1"/>
+<wire x1="21.465" y1="25.535" x2="22" y2="25" width="0.4064" layer="1"/>
+<wire x1="22" y1="25" x2="27" y2="25" width="0.4064" layer="1"/>
+<wire x1="27" y1="25" x2="28" y2="24" width="0.4064" layer="1"/>
+<wire x1="28" y1="24" x2="28" y2="19" width="0.4064" layer="1"/>
+<via x="28" y="19" extent="1-16" drill="0.6" shape="square"/>
+<wire x1="28" y1="19" x2="28" y2="13.4" width="0.4064" layer="16"/>
+<wire x1="28" y1="13.4" x2="26.6" y2="12" width="0.4064" layer="16"/>
+</signal>
 </signals>

Commit message: ROTARY_ENCODER + red led
Connections:
- removed net N$8: 3.3V.1, U1.VCC
- removed net ROTARY_C: ROTARY_C.1, U1.GPIO13
- net 3.3V: now also 3.3V.1, U1.VCC
- net GND: now also ROTARY_C.1
Routing:
- net N$8: track 49.3 -> 0.00 mm, vias 1 -> 0
- net 3.3V: track 21.1 -> 70.4 mm, vias 1 -> 2
- net ROTARY_C: track 35.5 -> 0.00 mm, vias 1 -> 0
- net GND: track 0.00 -> 32.3 mm, vias 17 -> 18
Changed lines of the file:
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@@
 <via x="30.29856875" y="2.900325" extent="1-16" drill="0.3048"/>
 <via x="3.599309375" y="11.4291625" extent="1-16" drill="0.3048"/>
+<contactref element="ROTARY_C" pad="1"/>
+<wire x1="8.618" y1="7.574" x2="13.22" y2="7.574" width="0.254" layer="1"/>
+<wire x1="13.22" y1="7.574" x2="13.92" y2="8.274" width="0.254" layer="1"/>
+<wire x1="13.92" y1="8.274" x2="13.92" y2="20.974" width="0.254" layer="1"/>
+<wire x1="13.92" y1="20.974" x2="14.047" y2="21.101" width="0.254" layer="1"/>
+<wire x1="14.047" y1="21.101" x2="26.747" y2="21.101" width="0.254" layer="1"/>
+<via x="26.747" y="21.101" extent="1-16" drill="0.3048"/>
+<wire x1="26.747" y1="21.101" x2="27.572" y2="21.926" width="0.254" layer="16"/>
+<wire x1="36.593753125" y1="36.133278125" x2="37" y2="45" width="0" layer="19" extent="1-1"/>
+<wire x1="29.56361875" y1="32.46638125" x2="36.593753125" y2="36.133278125" width="0" layer="19" extent="1-1"/>
+<wire x1="23.465" y1="27.83" x2="29.56361875" y2="32.46638125" width="0" layer="19" extent="1-1"/>
+<wire x1="27.572" y1="21.926" x2="23.465" y2="27.83" width="0" layer="19" extent="16-16"/>
+<wire x1="13.836" y1="5.417" x2="13.22" y2="7.574" width="0" layer="19" extent="1-16"/>
+<wire x1="29.347209375" y1="19.653046875" x2="27.572" y2="21.926" width="0" layer="19" extent="16-16"/>
+<wire x1="15.136" y1="2.692" x2="13.836" y2="5.417" width="0" layer="19" extent="16-16"/>
+<wire x1="12.978" y1="2.084" x2="15.136" y2="2.692" width="0" layer="19" extent="1-16"/>
+<wire x1="11.451" y1="2.692" x2="12.978" y2="2.084" width="0" layer="19" extent="1-16"/>
+<wire x1="31.967590625" y1="17.4788875" x2="29.347209375" y2="19.653046875" width="0" layer="19" extent="1-1"/>
+<wire x1="29.664" y1="15.342" x2="31.967590625" y2="17.4788875" width="0" layer="19" extent="1-1"/>
+<wire x1="26.997" y1="15.342" x2="29.664" y2="15.342" width="0" layer="19" extent="1-1"/>
+<wire x1="18.821" y1="2.692" x2="15.136" y2="2.692" width="0" layer="19" extent="16-16"/>
+<wire x1="17.3140125" y1="17.61843125" x2="14.047" y2="21.101" width="0" layer="19" extent="1-1"/>
+<wire x1="16.79455625" y1="15.0644375" x2="17.3140125" y2="17.61843125" width="0" layer="19" extent="1-1"/>
+<wire x1="11.557103125" y1="25.756665625" x2="14.047" y2="21.101" width="0" layer="19" extent="1-1"/>
+<wire x1="8.618" y1="21.194" x2="13.92" y2="20.974" width="0" layer="19" extent="1-1"/>
+<wire x1="4.11198125" y1="22.423528125" x2="8.618" y2="21.194" width="0" layer="19" extent="1-1"/>
+<wire x1="23.633659375" y1="11.211765625" x2="26.997" y2="15.342" width="0" layer="19" extent="1-1"/>
+<wire x1="4" y1="4" x2="8.618" y2="7.574" width="0" layer="19" extent="1-1"/>
+<wire x1="3.599309375" y1="11.4291625" x2="8.618" y2="7.574" width="0" layer="19" extent="1-1"/>
+<wire x1="29.572" y1="8.652" x2="23.633659375" y2="11.211765625" width="0" layer="19" extent="16-16"/>
+<wire x1="27.324" y1="5.654" x2="29.572" y2="8.652" width="0" layer="19" extent="1-16"/>
+<wire x1="30.29856875" y1="2.900325" x2="27.324" y2="5.654" width="0" layer="19" extent="1-1"/>
+<wire x1="33.508" y1="2.032" x2="30.29856875" y2="2.900325" width="0" layer="19" extent="1-1"/>
+<wire x1="35.4718625" y1="25.88095" x2="29.347209375" y2="19.653046875" width="0" layer="19" extent="1-1"/>
+<wire x1="15.106496875" y1="36.232490625" x2="11.557103125" y2="25.756665625" width="0" layer="19" extent="1-1"/>
+<wire x1="17.465" y1="42.83" x2="15.106496875" y2="36.232490625" width="0" layer="19" extent="1-1"/>
+<wire x1="10.86451875" y1="46.621753125" x2="17.465" y2="42.83" width="0" layer="19" extent="1-1"/>
+<wire x1="3.335934375" y1="39.769640625" x2="10.86451875" y2="46.621753125" width="0" layer="19" extent="1-1"/>
 </signal>
 <signal name="N$7">
@@
 <wire x1="25.572" y1="11.928" x2="25.572" y2="8.652" width="0.254" layer="16"/>
 </signal>
-<signal name="ROTARY_C">
-<contactref element="U1" pad="GPIO13"/>
-<contactref element="ROTARY_C" pad="1"/>
-<wire x1="8.618" y1="7.574" x2="13.22" y2="7.574" width="0.254" layer="1"/>
-<wire x1="13.22" y1="7.574" x2="13.92" y2="8.274" width="0.254" layer="1"/>
-<wire x1="13.92" y1="8.274" x2="13.92" y2="20.974" width="0.254" layer="1"/>
-<wire x1="13.92" y1="20.974" x2="14.047" y2="21.101" width="0.254" layer="1"/>
-<wire x1="14.047" y1="21.101" x2="26.747" y2="21.101" width="0.254" layer="1"/>
-<via x="26.747" y="21.101" extent="1-16" drill="0.3048"/>
-<wire x1="26.747" y1="21.101" x2="27.572" y2="21.926" width="0.254" layer="16"/>
-<wire x1="27.572" y1="21.926" x2="27.572" y2="25.052" width="0.254" layer="16"/>
-</signal>
 <signal name="ROTARY_A">
 <contactref element="U1" pad="GPIO14"/>
@@
 <wire x1="16.020365625" y1="22.401275" x2="19.421809375" y2="22.401275" width="0.254" layer="16"/>
 <wire x1="19.421809375" y1="22.401275" x2="19.572" y2="22.251084375" width="0.254" layer="16"/>
+<contactref element="U1" pad="VCC"/>
+<contactref element="3.3V" pad="1"/>
+<wire x1="8.554" y1="4.354" x2="8.5" y2="4.408" width="0.254" layer="1"/>
+<wire x1="8.5" y1="4.408" x2="8.5" y2="5.8" width="0.254" layer="1"/>
+<via x="8.5" y="5.8" extent="1-16" drill="0.3048"/>
+<wire x1="8.5" y1="5.8" x2="8.5" y2="29.1" width="0.254" layer="16"/>
+<wire x1="8.5" y1="29.1" x2="8.7" y2="29.3" width="0.254" layer="16"/>
+<wire x1="8.7" y1="29.3" x2="28.1" y2="29.3" width="0.254" layer="16"/>
+<wire x1="28.1" y1="29.3" x2="29.572" y2="27.828" width="0.254" layer="16"/>
+<wire x1="29.572" y1="27.828" x2="29.572" y2="25.052" width="0.254" layer="16"/>
+<wire x1="8.7" y1="29.3" x2="15.572" y2="25.052" width="0" layer="19" extent="16-16"/>
 </signal>
 <signal name="N$5">
@@
 <wire x1="24.77" y1="5.6" x2="24.824" y2="5.654" width="0.254" layer="1"/>
 </signal>
-<signal name="N$8">
-<contactref element="U1" pad="VCC"/>
-<contactref element="3.3V" pad="1"/>
-<wire x1="8.554" y1="4.354" x2="8.5" y2="4.408" width="0.254" layer="1"/>
-<wire x1="8.5" y1="4.408" x2="8.5" y2="5.8" width="0.254" layer="1"/>
-<via x="8.5" y="5.8" extent="1-16" drill="0.3048"/>
-<wire x1="8.5" y1="5.8" x2="8.5" y2="29.1" width="0.254" layer="16"/>
-<wire x1="8.5" y1="29.1" x2="8.7" y2="29.3" width="0.254" layer="16"/>
-<wire x1="8.7" y1="29.3" x2="28.1" y2="29.3" width="0.254" layer="16"/>
-<wire x1="28.1" y1="29.3" x2="29.572" y2="27.828" width="0.254" layer="16"/>
-<wire x1="29.572" y1="27.828" x2="29.572" y2="25.052" width="0.254" layer="16"/>
-</signal>
 <signal name="RX">

Commit message: EAGLE: resistance value update
Parts:
- R1: value 100 -> 250
- R2: value 100 -> 347
Changed lines of the file:
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@@
 <attribute name="NAME" x="2.0644125" y="12.1147375" size="0.6096" layer="25"/>
 </element>
-<element name="R1" library="rcl" package="R0603" value="100" x="19.508" y="13.354" smashed="yes" rot="R90">
+<element name="R1" library="rcl" package="R0603" value="250" x="19.508" y="13.354" smashed="yes" rot="R90">
 <attribute name="NAME" x="18.873" y="12.719" size="0.6096" layer="25" rot="R90"/>
 <attribute name="VALUE" x="21.413" y="12.719" size="1.27" layer="27" rot="R90"/>
 </element>
-<element name="R2" library="rcl" package="R0603" value="100" x="21.54" y="13.354" smashed="yes" rot="R90">
+<element name="R2" library="rcl" package="R0603" value="347" x="21.54" y="13.354" smashed="yes" rot="R90">
 <attribute name="NAME" x="20.905" y="12.719" size="0.6096" layer="25" rot="R90"/>
 <attribute name="VALUE" x="23.445" y="12.719" size="1.27" layer="27" rot="R90"/>
